File: LEDLamp_CapTIvate.brd (EAGLE design)
At the start: 50.1 x 100 mm, 8 parts, among them Q1 IRLL024N, Q2 IRLL024N

Commit message: V1.1
Parts:
- added 12V, CW12V, CWIN, GND, WW12V, WWIN: (no value), wirepad:SMD2,54-5,08
- added C1: 2.2n, rcl:C0805
- added C2, C5: 100n, rcl:C0805
- added C3: 10u, rcl:R/2012-12R
- added C4: 330n, rcl:C0805
- added IC1: UA78M33, MSP430_Lab:SOT223
- added JTAG_: MSP430SBWMPE, GG_JTAG:MPE-374-04
- added R5: 47k, rcl:R0805
- added U$2: OSHW_LOGO_SYMM, PatternAgents-Logos:OSHW_LOGO_MED_SYM
- added U$6: (no value), Piktogramme:BUCH1
- added U$7: (no value), Piktogramme:LUPE1
- added U$8: (no value), Piktogramme:TASSE1
- moved R2 104.8 mm to (25.3, 79.4), flipped to the bottom
- moved Q2 99.2 mm to (18.9, 82.8), flipped to the bottom
- moved R1 96.7 mm to (42.1, 79.4), flipped to the bottom
- moved Q1 91.9 mm to (31.2, 82.7), flipped to the bottom
- moved U$3 53.5 mm to (50.4, 10.3), turned to 90 degrees
Connections:
- new net RST: C1.1, JTAG_.P$3, R5.1, U$1.5
- new net RX: U$1.8
- new net TST: JTAG_.P$4, U$1.6
- new net TX: U$1.7
- new net VCC: 12V.1, C4.2, CW12V.1, IC1.1, WW12V.1
- new net VCCINT: C2.1, C3.+, C5.2, IC1.3, JTAG_.P$1, R5.2, U$1.4
- net GND: now also C1.2, C2.2, C3.-, C4.1, C5.1, GND.1, IC1.2, JTAG_.P$2, U$1.3
- net N$11: now also WWIN.1
- net N$12: now also CWIN.1
Routing:
- net N$5: track 0.00 -> 128.0 mm
- net GND: track 0.00 -> 117.0 mm
- net N$1: track 0.00 -> 99.2 mm, vias 0 -> 4
- net VCC: track 0.00 -> 95.3 mm
- net WW: track 0.00 -> 64.7 mm
- net CW: track 0.00 -> 52.5 mm
- net VCCINT: track 0.00 -> 37.6 mm
- net N$6: track 0.00 -> 29.1 mm
- net N$8: track 0.00 -> 29.0 mm
- net N$4: track 0.00 -> 27.5 mm
- net N$2: track 0.00 -> 24.5 mm
- net TST: track 0.00 -> 17.0 mm
- net RST: track 0.00 -> 12.7 mm
- net N$3: track 0.00 -> 11.3 mm, vias 0 -> 1
- net N$7: track 0.00 -> 9.24 mm
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- added copper zone on layer 1, net N$13
- removed copper zone on layer 1, net GND
Other:
- board size 50.1 x 100 mm -> 50 x 100 mm
- board text added: "12V"
- board text added: "LED1"
- board text added: "LED2"
- board text added: "V1.1"

Commit message: V1.2
Parts:
- added C6: 1u, rcl:R/2012-12R
- added LED1, LED2, LED3: (no value), led:MINI-TOPLED-SANTANA
- added PAD1, PAD2: WIREPADSMD1,27-254, wirepad:SMD3X1.5
- added R3, R4, R6: 47k, rcl:R0805
- moved 12V 3.06 mm to (12.0, 87.3)
- moved GND 2.55 mm to (15.5, 87.3)
- moved Q2 1.00 mm to (19.9, 82.8)
- moved U$6 1.00 mm to (7.43, 87.6)
- moved WW12V 1.00 mm to (24.0, 91.0)
- moved WWIN 1.00 mm to (20.0, 91.0)
- moved U$3 0.90 mm to (49.5, 10.4)
- renumbered U$1 to MSP430FR2633
Connections:
- new net N$14: LED3.A, R6.1
- new net N$15: LED2.A, R4.1
- new net N$16: LED1.A, R3.1
- new net N$18: MSP430FR2633.11, R3.2
- new net N$19: MSP430FR2633.10, R4.2
- new net N$20: MSP430FR2633.9, R6.2
- new net N$21: C6.+, MSP430FR2633.24
- net GND: now also C6.-, LED1.C, LED2.C, LED3.C
- net RX: now also PAD2.P$1
- net TX: now also PAD1.P$1
Routing:
- net N$14: track 0.00 -> 126.2 mm
- net GND: track 117.0 -> 217.7 mm, vias 0 -> 4
- net N$15: track 0.00 -> 71.7 mm
- net N$16: track 0.00 -> 35.4 mm
- net N$20: track 0.00 -> 33.8 mm, vias 0 -> 2
- net N$19: track 0.00 -> 31.3 mm, vias 0 -> 2
- net N$18: track 0.00 -> 29.3 mm, vias 0 -> 2
- net N$21: track 0.00 -> 22.2 mm, vias 0 -> 2
- net RX: track 0.00 -> 17.6 mm
- net TX: track 0.00 -> 13.4 mm
- net N$5: track 128.0 -> 120.7 mm
- net N$6: track 29.1 -> 23.5 mm
- net N$10: track 3.15 -> 2.15 mm
Other:
- board text added: "2016"
- board text added: "V1.2"
- board text removed: "V1.1"

Commit message: V1.3
Parts:
- moved R2 17.9 mm to (43.0, 77.3)
- moved R1 1.00 mm to (43.1, 79.4)
- moved U$7 0.38 mm to (9.32, 46.1)
- moved U$8 0.25 mm to (9.40, 4.76)
- moved U$6 0.13 mm to (7.43, 87.7)
Routing:
- net N$10: track 2.15 -> 20.9 mm
- net WW: track 64.7 -> 48.7 mm
- net N$21: track 22.2 -> 20.4 mm
- net N$9: track 7.76 -> 8.67 mm
Other:
- board text added: "V1.3"
- board text removed: "V1.2"
