File: LEDLamp_CapTIvate.sch (EAGLE design)
At the start: 7 parts, among them Q1 IRLL024N, Q2 IRLL024N

Commit message: V1.1
Parts:
- added 12V, CW12V, CWIN, GND, WW12V, WWIN: (no value), wirepad:SMD5
- added C1: 2.2n, rcl:C-EUC0805
- added C2, C5: 100n, rcl:C-EUC0805
- added C3: 10u, rcl:CPOL-EUR/2012-12R
- added C4: 330n, rcl:C-EUC0805
- added IC1: UA78M33, MSP430_Lab:UA78M05DCY
- added JTAG_: MSP430SBWMPE, GG_JTAG:MSP430SBWMPE
- added R5: 47k, rcl:R-EU_R0805
- added U$2: OSHW_LOGO_SYMM, PatternAgents-Logos:OSHW_LOGO_SYMM
Connections:
- new net RST: C1.1, JTAG_RST.S, R5.1, U$1.#RST/NMI/SBWTDIO
- new net RX: U$1.P1.5/UCA0RXD/UCA0SOMI/TA1.1/TMS/A5
- new net TST: JTAG_TST.S, U$1.TEST/SBWTCK
- new net TX: U$1.P1.4/UCA0TXD/UCA0SIMO/TA1.2/TCK/A4/VREF+
- new net VCC: 12V.P, C4.2, CW12V.P, IC1.IN, WW12V.P
- new net VCCINT: C2.1, C3.+, C5.2, IC1.OUT, JTAG_VCC.S, R5.2, U$1.DVCC
- net GND: now also C1.2, C2.2, C3.-, C4.1, C5.1, GND.P, IC1.GND, JTAG_GND.S, U$1.DVSS
- net N$11: now also WWIN.P
- net N$12: now also CWIN.P
Other:
- moved on the sheet: Q1, Q2, R1, R2

Commit message: V1.2
Parts:
- added C6: 1u, rcl:CPOL-EUR/2012-12R
- added LED1, LED2, LED3: (no value), led:LEDTOPLED-SANTANA
- added PAD1, PAD2: WIREPADSMD1,27-254, wirepad:WIREPADSMD3X1,5
- added R3, R4, R6: 47k, rcl:R-EU_R0805
- renumbered U$1 to MSP430FR2633
Connections:
- new net N$14: LED3.A, R6.1
- new net N$15: LED2.A, R4.1
- new net N$16: LED1.A, R3.1
- new net N$18: MSP430FR2633.P1.0/UCB0STE/TA0CLK/A0/VEREF+, R3.2
- new net N$19: MSP430FR2633.P1.7/UCA0STE/SMCLK/TDO/A7, R4.2
- new net N$20: MSP430FR2633.P1.6/UCA0CLK/TA1CLK/TDI/TCLK/A6, R6.2
- new net N$21: C6.+, MSP430FR2633.VREG
- net GND: now also C6.-, LED1.C, LED2.C, LED3.C
- net RX: now also PAD2.P
- net TX: now also PAD1.P
Other:
- moved on the sheet: C1, R5
